File: esplog_ldo/esplog_ldo.kicad_pcb (KiCad board)
At the start: 2 copper layers, 13.5 x 10.7 mm, 28 parts, among them SW1 SW_Push, U1 ESP32-C3, U2 BMI160, U3 SPX3819M5-L-3-3, Y1 Crystal_GND24

Commit message: Add component values
Parts:
- C1, C2: value C -> 10p
- C10: value C -> 20n
- C11, C4, C6, C8, C9: value C -> 100n
- C3: value C -> 1u
- C5: value C -> 4.7u
- C7: value C -> 22u
- R1: value R -> 10k
- U2: value BMI160 -> BMI270
- Y1: value Crystal_GND24 -> 40M
Other:
- board text added: "BMI270 C3"
- board text removed: "BMI160 C3"
Changed lines of the file:
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@@
       (effects (font (size 1 1) (thickness 0.15)))
     )
-    (fp_text value "C" (at 0 1.16 90) (layer "F.Fab") hide
+    (fp_text value "100n" (at 0 1.16 90) (layer "F.Fab") hide
       (effects (font (size 1 1) (thickness 0.15)))
     )
@@
       (effects (font (size 1 1) (thickness 0.15)))
     )
-    (fp_text value "C" (at 0 1.16 90) (layer "F.Fab") hide
+    (fp_text value "10p" (at 0 1.16 90) (layer "F.Fab") hide
       (effects (font (size 1 1) (thickness 0.15)))
     )
@@
       (effects (font (size 1 1) (thickness 0.15)))
     )
-    (fp_text value "C" (at 0 1.16 90) (layer "F.Fab") hide
+    (fp_text value "100n" (at 0 1.16 90) (layer "F.Fab") hide
       (effects (font (size 1 1) (thickness 0.15)))
     )
@@
       (effects (font (size 1 1) (thickness 0.15)))
     )
-    (fp_text value "C" (at 0 1.16) (layer "F.Fab") hide
+    (fp_text value "100n" (at 0 1.16) (layer "F.Fab") hide
       (effects (font (size 1 1) (thickness 0.15)))
     )
@@
       (effects (font (size 1 1) (thickness 0.15)))
     )
-    (fp_text value "C" (at 0 1.16) (layer "F.Fab") hide
+    (fp_text value "100n" (at 0 1.16) (layer "F.Fab") hide
       (effects (font (size 1 1) (thickness 0.15)))
     )
@@
       (effects (font (size 1 1) (thickness 0.15)))
     )
-    (fp_text value "C" (at 0 1.16 90) (layer "F.Fab") hide
+    (fp_text value "10p" (at 0 1.16 90) (layer "F.Fab") hide
       (effects (font (size 1 1) (thickness 0.15)))
     )
@@
       (effects (font (size 1 1) (thickness 0.15)))
     )
-    (fp_text value "C" (at 0 1.43 90) (layer "F.Fab") hide
+    (fp_text value "22u" (at 0 1.43 90) (layer "F.Fab") hide
       (effects (font (size 1 1) (thickness 0.15)))
     )
@@
       (effects (font (size 1 1) (thickness 0.15)))
     )
-    (fp_text value "BMI160" (at 0 2.5 90) (layer "F.Fab") hide
+    (fp_text value "BMI270" (at 0 2.5 90) (layer "F.Fab") hide
       (effects (font (size 1 1) (thickness 0.15)))
     )
@@
       (effects (font (size 1 1) (thickness 0.15)))
     )
-    (fp_text value "C" (at 0 1.16 90) (layer "F.Fab") hide
+    (fp_text value "100n" (at 0 1.16 90) (layer "F.Fab") hide
       (effects (font (size 1 1) (thickness 0.15)))
     )
@@
       (effects (font (size 1 1) (thickness 0.15)))
     )
-    (fp_text value "C" (at 0 1.43) (layer "F.Fab")
+    (fp_text value "4.7u" (at 0 1.43) (layer "F.Fab")
       (effects (font (size 1 1) (thickness 0.15)))
     )
@@
       (effects (font (size 1 1) (thickness 0.15)))
     )
-    (fp_text value "Crystal_GND24" (at 0 2.45) (layer "F.Fab") hide
+    (fp_text value "40M" (at 0 2.45) (layer "F.Fab") hide
       (effects (font (size 1 1) (thickness 0.15)))
     )
@@
       (effects (font (size 1 1) (thickness 0.15)))
     )
-    (fp_text value "C" (at 0 1.16 90) (layer "F.Fab") hide
+    (fp_text value "1u" (at 0 1.16 90) (layer "F.Fab") hide
       (effects (font (size 1 1) (thickness 0.15)))
     )
@@
       (effects (font (size 1 1) (thickness 0.15)))
     )
-    (fp_text value "R" (at 0 1.17 90) (layer "F.Fab") hide
+    (fp_text value "10k" (at 0 1.17 90) (layer "F.Fab") hide
       (effects (font (size 1 1) (thickness 0.15)))
     )
@@
       (effects (font (size 1 1) (thickness 0.15)))
     )
-    (fp_text value "C" (at 0 1.16 90) (layer "F.Fab") hide
+    (fp_text value "20n" (at 0 1.16 90) (layer "F.Fab") hide
       (effects (font (size 1 1) (thickness 0.15)))
     )
@@
   )
   (gr_rect (start 82.6516 53.7464) (end 96.1644 64.4652) (layer "Edge.Cuts") (width 0.1) (fill none))
-  (gr_text "BMI160 C3" (at 93.0148 60.0456 270) (layer "B.SilkS")
+  (gr_text "BMI270 C3" (at 93.0148 60.0456 270) (layer "B.SilkS")
     (effects (font (size 1 1) (thickness 0.15)) (justify mirror))
   )
