File: esplog_ldo/esplog_ldo.kicad_sch (KiCad schematic)
At the start: 27 parts, among them SW1 SW_Push, U1 ESP32-C3, U2 BMI160, U3 SPX3819M5-L-3-3, Y1 Crystal_GND24

Commit message: Add component values
Parts:
- C1, C2: value C -> 10p
- C10: value C -> 20n
- C11, C4, C6, C8, C9: value C -> 100n
- C3: value C -> 1u
- C5: value C -> 4.7u
- C7: value C -> 22u
- R1: value R -> 10k
- U2: value BMI160 -> BMI270
- Y1: value Crystal_GND24 -> 40M
Other:
- moved on the sheet: C7, C8
Changed lines of the file:
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@@
       (effects (font (size 1.27 1.27)) (justify left))
     )
-    (property "Value" "R" (id 1) (at 100.33 134.6199 0)
+    (property "Value" "10k" (id 1) (at 100.33 134.6199 0)
       (effects (font (size 1.27 1.27)) (justify left))
     )
@@
     (pin "1")
   )
-  (symbol (lib_id "Device:C") (at 106.68 160.02 180) (unit 1)
-    (in_bom yes) (on_board yes)
-    (property "Reference" "C8" (id 0) (at 104.14 157.48 90))
-    (property "Value" "C" (id 1) (at 104.14 162.56 90))
-    (property "Footprint" "Capacitor_SMD:C_0402_1005Metric" (id 2) (at 105.7148 156.21 0)
-      (effects (font (size 1.27 1.27)) hide)
-    )
-    (property "Datasheet" "~" (id 3) (at 106.68 160.02 0)
+  (symbol (lib_id "Device:C") (at 100.33 160.02 180) (unit 1)
+    (in_bom yes) (on_board yes)
+    (property "Reference" "C8" (id 0) (at 97.79 157.48 90))
+    (property "Value" "100n" (id 1) (at 97.79 162.56 90))
+    (property "Footprint" "Capacitor_SMD:C_0402_1005Metric" (id 2) (at 99.3648 156.21 0)
+      (effects (font (size 1.27 1.27)) hide)
+    )
+    (property "Datasheet" "~" (id 3) (at 100.33 160.02 0)
       (effects (font (size 1.27 1.27)) hide)
     )
@@
     (in_bom yes) (on_board yes)
     (property "Reference" "C11" (id 0) (at 85.09 157.48 90))
-    (property "Value" "C" (id 1) (at 85.09 162.56 90))
+    (property "Value" "100n" (id 1) (at 85.09 162.56 90))
     (property "Footprint" "Capacitor_SMD:C_0402_1005Metric" (id 2) (at 86.6648 156.21 0)
       (effects (font (size 1.27 1.27)) hide)
@@
     (pin "2")
   )
-  (symbol (lib_id "Device:C") (at 100.33 160.02 180) (unit 1)
-    (in_bom yes) (on_board yes)
-    (property "Reference" "C7" (id 0) (at 97.79 157.48 90))
-    (property "Value" "C" (id 1) (at 97.79 162.56 90))
-    (property "Footprint" "Capacitor_SMD:C_0603_1608Metric" (id 2) (at 99.3648 156.21 0)
-      (effects (font (size 1.27 1.27)) hide)
-    )
-    (property "Datasheet" "~" (id 3) (at 100.33 160.02 0)
+  (symbol (lib_id "Device:C") (at 106.68 160.02 180) (unit 1)
+    (in_bom yes) (on_board yes)
+    (property "Reference" "C7" (id 0) (at 104.14 157.48 90))
+    (property "Value" "22u" (id 1) (at 104.14 162.56 90))
+    (property "Footprint" "Capacitor_SMD:C_0603_1608Metric" (id 2) (at 105.7148 156.21 0)
+      (effects (font (size 1.27 1.27)) hide)
+    )
+    (property "Datasheet" "~" (id 3) (at 106.68 160.02 0)
       (effects (font (size 1.27 1.27)) hide)
     )
@@
       (effects (font (size 1.27 1.27)) (justify left))
     )
-    (property "Value" "BMI160" (id 1) (at 240.7794 101.6 0)
+    (property "Value" "BMI270" (id 1) (at 240.7794 101.6 0)
       (effects (font (size 1.27 1.27)) (justify left))
     )
@@
     (in_bom yes) (on_board yes)
     (property "Reference" "Y1" (id 0) (at 101.6 63.5 90))
-    (property "Value" "Crystal_GND24" (id 1) (at 102.87 66.04 90))
+    (property "Value" "40M" (id 1) (at 102.87 66.04 90))
     (property "Footprint" "Crystal:Crystal_SMD_3225-4Pin_3.2x2.5mm" (id 2) (at 101.6 71.12 0)
       (effects (font (size 1.27 1.27)) hide)
@@
     (in_bom yes) (on_board yes)
     (property "Reference" "C6" (id 0) (at 91.44 157.48 90))
-    (property "Value" "C" (id 1) (at 91.44 162.56 90))
+    (property "Value" "100n" (id 1) (at 91.44 162.56 90))
     (property "Footprint" "Capacitor_SMD:C_0402_1005Metric" (id 2) (at 93.0148 156.21 0)
       (effects (font (size 1.27 1.27)) hide)
@@
     (in_bom yes) (on_board yes)
     (property "Reference" "C4" (id 0) (at 100.33 99.06 90))
-    (property "Value" "C" (id 1) (at 95.25 99.06 90))
+    (property "Value" "100n" (id 1) (at 95.25 99.06 90))
     (property "Footprint" "Capacitor_SMD:C_0402_1005Metric" (id 2) (at 101.6 100.6348 0)
       (effects (font (size 1.27 1.27)) hide)
@@
     (in_bom yes) (on_board yes)
     (property "Reference" "C2" (id 0) (at 93.98 72.39 90))
-    (property "Value" "C" (id 1) (at 88.9 72.39 90))
+    (property "Value" "10p" (id 1) (at 88.9 72.39 90))
     (property "Footprint" "Capacitor_SMD:C_0402_1005Metric" (id 2) (at 95.25 73.9648 0)
       (effects (font (size 1.27 1.27)) hide)
@@
     (in_bom yes) (on_board yes)
     (property "Reference" "C1" (id 0) (at 93.98 64.77 90))
-    (property "Value" "C" (id 1) (at 88.9 64.77 90))
+    (property "Value" "10p" (id 1) (at 88.9 64.77 90))
     (property "Footprint" "Capacitor_SMD:C_0402_1005Metric" (id 2) (at 95.25 66.3448 0)
       (effects (font (size 1.27 1.27)) hide)
@@
     (in_bom yes) (on_board yes)
     (property "Reference" "C9" (id 0) (at 179.07 91.44 90))
-    (property "Value" "C" (id 1) (at 184.15 91.44 90))
+    (property "Value" "100n" (id 1) (at 184.15 91.44 90))
     (property "Footprint" "Capacitor_SMD:C_0402_1005Metric" (id 2) (at 177.8 89.8652 0)
       (effects (font (size 1.27 1.27)) hide)
@@
     (in_bom yes) (on_board yes)
     (property "Reference" "C3" (id 0) (at 93.98 134.62 90))
-    (property "Value" "C" (id 1) (at 88.9 134.62 90))
+    (property "Value" "1u" (id 1) (at 88.9 134.62 90))
     (property "Footprint" "Capacitor_SMD:C_0402_1005Metric" (id 2) (at 95.25 136.1948 0)
       (effects (font (size 1.27 1.27)) hide)
@@
     (in_bom yes) (on_board yes)
     (property "Reference" "C10" (id 0) (at 152.4 147.32 90))
-    (property "Value" "C" (id 1) (at 152.4 152.4 90))
+    (property "Value" "20n" (id 1) (at 152.4 152.4 90))
     (property "Footprint" "Capacitor_SMD:C_0402_1005Metric" (id 2) (at 153.9748 146.05 0)
       (effects (font (size 1.27 1.27)) hide)
@@
     (in_bom yes) (on_board yes)
     (property "Reference" "C5" (id 0) (at 137.16 147.32 90))
-    (property "Value" "C" (id 1) (at 137.16 152.4 90))
+    (property "Value" "4.7u" (id 1) (at 137.16 152.4 90))
     (property "Footprint" "Capacitor_SMD:C_0603_1608Metric" (id 2) (at 138.7348 146.05 0)
       (effects (font (size 1.27 1.27)) hide)
@@
     )
     (path "/a9556758-e492-4822-bd4e-a08b0a5efbf3"
-      (reference "C1") (unit 1) (value "C") (footprint "Capacitor_SMD:C_0402_1005Metric")
+      (reference "C1") (unit 1) (value "10p") (footprint "Capacitor_SMD:C_0402_1005Metric")
     )
     (path "/998e2bb4-6515-4e6a-8bf9-65b9dac782a0"
-      (reference "C2") (unit 1) (value "C") (footprint "Capacitor_SMD:C_0402_1005Metric")
+      (reference "C2") (unit 1) (value "10p") (footprint "Capacitor_SMD:C_0402_1005Metric")
     )
     (path "/b0061c6b-e8c7-4f80-b07f-9febe7a410d4"
-      (reference "C3") (unit 1) (value "C") (footprint "Capacitor_SMD:C_0402_1005Metric")
+      (reference "C3") (unit 1) (value "1u") (footprint "Capacitor_SMD:C_0402_1005Metric")
     )
     (path "/9814b1e2-94b2-4a42-b7b9-8afdf2af0d80"
-      (reference "C4") (unit 1) (value "C") (footprint "Capacitor_SMD:C_0402_1005Metric")
+      (reference "C4") (unit 1) (value "100n") (footprint "Capacitor_SMD:C_0402_1005Metric")
     )
     (path "/cbf9915d-29be-43a2-8a15-02fe3d77325e"
-      (reference "C5") (unit 1) (value "C") (footprint "Capacitor_SMD:C_0603_1608Metric")
+      (reference "C5") (unit 1) (value "4.7u") (footprint "Capacitor_SMD:C_0603_1608Metric")
     )
     (path "/80e8e45c-35b4-4460-b2aa-ee9691244466"
-      (reference "C6") (unit 1) (value "C") (footprint "Capacitor_SMD:C_0402_1005Metric")
+      (reference "C6") (unit 1) (value "100n") (footprint "Capacitor_SMD:C_0402_1005Metric")
     )
     (path "/5b8a528b-5486-481d-a344-872a071296a3"
-      (reference "C7") (unit 1) (value "C") (footprint "Capacitor_SMD:C_0603_1608Metric")
+      (reference "C7") (unit 1) (value "22u") (footprint "Capacitor_SMD:C_0603_1608Metric")
     )
     (path "/31a740e6-bcb7-45db-8e0b-ce4e6ba60fd0"
-      (reference "C8") (unit 1) (value "C") (footprint "Capacitor_SMD:C_0402_1005Metric")
+      (reference "C8") (unit 1) (value "100n") (footprint "Capacitor_SMD:C_0402_1005Metric")
     )
     (path "/ac7711a6-1dae-41b8-8378-b5d561d56c0d"
-      (reference "C9") (unit 1) (value "C") (footprint "Capacitor_SMD:C_0402_1005Metric")
+      (reference "C9") (unit 1) (value "100n") (footprint "Capacitor_SMD:C_0402_1005Metric")
     )
     (path "/c8c1c818-ba84-4392-8206-b3f1c777de07"
-      (reference "C10") (unit 1) (value "C") (footprint "Capacitor_SMD:C_0402_1005Metric")
+      (reference "C10") (unit 1) (value "20n") (footprint "Capacitor_SMD:C_0402_1005Metric")
     )
     (path "/3a74b789-01f2-4da3-b288-5c94df937773"
-      (reference "C11") (unit 1) (value "C") (footprint "Capacitor_SMD:C_0402_1005Metric")
+      (reference "C11") (unit 1) (value "100n") (footprint "Capacitor_SMD:C_0402_1005Metric")
     )
     (path "/53dd8859-60b4-47dd-97d6-6a1156adc453"
@@
     )
     (path "/2b2fe637-ea9e-4be3-be9a-8483fb30adf5"
-      (reference "R1") (unit 1) (value "R") (footprint "Resistor_SMD:R_0402_1005Metric")
+      (reference "R1") (unit 1) (value "10k") (footprint "Resistor_SMD:R_0402_1005Metric")
     )
     (path "/f1886dad-5860-43b2-b743-d26e60afbe12"
@@
     )
     (path "/61df5b74-84d3-48ee-9418-823388748e83"
-      (reference "U2") (unit 1) (value "BMI160") (footprint "Package_LGA:Bosch_LGA-14_3x2.5mm_P0.5mm")
+      (reference "U2") (unit 1) (value "BMI270") (footprint "Package_LGA:Bosch_LGA-14_3x2.5mm_P0.5mm")
     )
     (path "/f7249b16-acdb-41c5-8809-c3b8edb7e35c"
@@
     )
     (path "/72d0e0a0-ba3a-4196-962b-e772ebd4e701"
-      (reference "Y1") (unit 1) (value "Crystal_GND24") (footprint "Crystal:Crystal_SMD_3225-4Pin_3.2x2.5mm")
-    )
-  )
+      (reference "Y1") (unit 1) (value "40M") (footprint "Crystal:Crystal_SMD_3225-4Pin_3.2x2.5mm")
+    )
+  )
